File: X17_Pi_Shield.kicad_pcb (KiCad board)
At the start: 2 copper layers, 85 x 56 mm, 107 parts, among them J1 BM04B-GHS-TBT, J10 BM04B-GHS-TBT, J11 BM04B-GHS-TBT, J12 Conn_01x05_Pin, J13 Conn_01x03_Pin, J14 Conn_01x03_Pin, J19 430450212, J2 BM02B-GHS-TBT, J20 Conn_01x02_Pin, J21 Conn_01x02_Pin, J22 430450212, J23 430450612, J24 430450212, J3 BM02B-GHS-TBT, J4 BM02B-GHS-TBT, J5 BM02B-GHS-TBT, J6 Conn_01x03_Pin, J7 BM04B-GHS-TBT, J8 UJC-HP-L-G-5-MSMT-TR, J9 430450612, J9 Conn_01x04_Pin, U1 4754, U10 4754, U2 TPS2117DRLR, U3 INA260AIPW, U4 AZ1117IH-3.3TRG1, U5 MAX485, U6 MMBT3906LT3G, U7 ISOW1432BDFMR, U8 RASPBERRY_PI_4B_4GB, U9 ISO3086TDW

Commit message: Updating 3d Models
Parts:
- removed the C1 at (-5.63, -17.6)
- removed the C1 at (157.9, 49.7)
- removed the C10 at (157.9, 67.7)
- removed the C10 at (-1.28, -10.1)
- removed C11: 10nF, Capacitor_SMD:C_0805_2012Metric_Pad1.18x1.45mm_HandSolder
- removed the C2 at (-5.63, -15.1)
- removed the C2 at (157.9, 52.7)
- removed the C3 at (157.9, 55.7)
- removed the C3 at (-5.63, -12.6)
- removed the C7 at (157.9, 58.7)
- removed the C7 at (-1.28, -17.6)
- removed the C8 at (-1.28, -15.1)
- removed the C8 at (157.9, 61.7)
- removed the C9 at (157.9, 64.7)
- removed the C9 at (-1.28, -12.6)
- removed J19: 430450212, 0430450212/:CON_430450212_MOL
- removed the J9 at (171.7, 56.3)
- removed the J9 at (-2.88, 1.26)
- removed the R17 at (162.7, 79.8)
- removed the R17 at (3.07, -15.1)
- removed the R5 at (162.7, 62.1)
- removed the R5 at (-1.28, -7.56)
- removed R7, R8: 10k, Resistor_SMD:R_0805_2012Metric_Pad1.20x1.40mm_HandSolder
- removed the R9 at (3.07, -17.6)
- removed the R9 at (162.7, 70.9)
- removed the REF** at (38.8, 70.2)
- removed the REF** at (96.8, 70.2)
- removed the REF** at (96.8, 21.2)
- removed the REF** at (38.8, 21.2)
- removed U9: ISO3086TDW, ISO3086TDW:SOIC127P1030X265-16N
- added C1: 10uF, Capacitor_SMD:C_0603_1608Metric_Pad1.08x0.95mm_HandSolder, F.Cu at (73.2, 96.5)
- added C10: 0.1uF, Capacitor_SMD:C_0603_1608Metric_Pad1.08x0.95mm_HandSolder, F.Cu at (72.1, 88.5)
- added C2: 1uF, Capacitor_SMD:C_0603_1608Metric_Pad1.08x0.95mm_HandSolder, F.Cu at (69.8, 96.5)
- added C3: 10nF, Capacitor_SMD:C_0603_1608Metric_Pad1.08x0.95mm_HandSolder, F.Cu at (66.4, 96.5)
- added C7: 10nF, Capacitor_SMD:C_0603_1608Metric_Pad1.08x0.95mm_HandSolder, F.Cu at (89.9, 105.5)
- added C8: 0.1uF, Capacitor_SMD:C_0603_1608Metric_Pad1.08x0.95mm_HandSolder, F.Cu at (91.1, 87.3)
- added C9: 10uF, Capacitor_SMD:C_0603_1608Metric_Pad1.08x0.95mm_HandSolder, F.Cu at (94.9, 87.3)
- added J9: Conn_01x04_Pin, Connector_PinHeader_2.54mm:PinHeader_1x04_P2.54mm_Vertical, F.Cu at (230.0, 119.0)
- added R17: 120, Resistor_SMD:R_0603_1608Metric_Pad0.98x0.95mm_HandSolder, F.Cu at (91.5, 91.5)
- added R5: 120, Resistor_SMD:R_0603_1608Metric_Pad0.98x0.95mm_HandSolder, F.Cu at (40.7, 113.0)
- added R9: 5k, Resistor_SMD:R_0603_1608Metric_Pad0.98x0.95mm_HandSolder, F.Cu at (68.2, 88.5)
- added REF**: MountingHole_2.7mm_M2.5_ISO14580, MountingHole:MountingHole_2.7mm_M2.5_ISO14580, F.Cu at (104.0, 21.0)
- added REF**: MountingHole_2.7mm_M2.5_ISO14580, MountingHole:MountingHole_2.7mm_M2.5_ISO14580, F.Cu at (46.0, 70.0)
- added REF**: MountingHole_2.7mm_M2.5_ISO14580, MountingHole:MountingHole_2.7mm_M2.5_ISO14580, F.Cu at (104.0, 70.0)
- added REF**: MountingHole_2.7mm_M2.5_ISO14580, MountingHole:MountingHole_2.7mm_M2.5_ISO14580, F.Cu at (46.0, 21.0)
- U5: footprint AZ1117IH_3_3TRG1:SOT223_AZ1117I_6P5X3P5_DIO-M -> MAX485:SO08
- moved U8 219.2 mm to (236.2, 46.5)
- moved U4 194.9 mm to (87.5, 172.2)
- moved J8 184.8 mm to (21.5, 189.5)
- moved J14 182.8 mm to (275.3, 97.8)
- moved J22 174.6 mm to (110.8, 96.7)
- moved C15 170.9 mm to (261.5, 118.5)
- moved JP4 166.1 mm to (20.3, 172.8)
- moved U10 166.1 mm to (236.0, 97.2)
- moved C17 165.5 mm to (25.1, 172.2)
- moved C16 165.3 mm to (256.4, 125.0)
- moved U5 165.1 mm to (23.3, 112.4)
- moved JP3 165.0 mm to (20.5, 166.8)
- moved C13 164.6 mm to (255.6, 118.5)
- moved J11 164.2 mm to (259.2, 106.0)
- moved J10 164.1 mm to (258.8, 93.5)
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
Commit message: Added header and updated mounting pins
Parts:
- removed the REF** at (104.0, 21.0)
- removed the REF** at (46.0, 70.0)
- removed the REF** at (104.0, 70.0)
- removed the REF** at (46.0, 21.0)
- added REF**: MountingHole_2.7mm_M2.5_ISO14580, MountingHole:MountingHole_2.7mm_M2.5_ISO14580, F.Cu at (121.5, 119.0)
- added REF**: MountingHole_2.7mm_M2.5_ISO14580, MountingHole:MountingHole_2.7mm_M2.5_ISO14580, F.Cu at (179.5, 70.0)
- added REF**: MountingHole_2.7mm_M2.5_ISO14580, MountingHole:MountingHole_2.7mm_M2.5_ISO14580, F.Cu at (121.5, 70.0)
- added REF**: MountingHole_2.7mm_M2.5_ISO14580, MountingHole:MountingHole_2.7mm_M2.5_ISO14580, F.Cu at (179.5, 119.0)
- U8: footprint RASPBERRY_PI_4B_4GB:MODULE_RASPBERRY_PI_4B_4GB -> TSW-120-09-G-D:SAMTEC_TSW-120-09-G-D
- moved D1 100.7 mm to (52.6, 60.1)
- moved J1 100.7 mm to (51.6, 22.0)
- moved J2 100.7 mm to (34.0, 35.2)
- moved J3 100.7 mm to (33.8, 44.7)
- moved J4 100.7 mm to (33.1, 54.4)
- moved J5 100.7 mm to (33.0, 64.2)
- moved J6 100.7 mm to (53.9, 45.1)
- moved J7 100.7 mm to (37.4, 22.2)
- moved R1 100.7 mm to (44.2, 42.1)
- moved R2 100.7 mm to (44.2, 44.6)
- moved R3 100.7 mm to (44.2, 47.1)
- moved R4 100.7 mm to (44.2, 49.6)
- moved U6 100.7 mm to (46.4, 54.4)
- moved C6 79.5 mm to (138.6, 163.8)
- moved C8 79.5 mm to (139.3, 150.5)
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
Commit message: Initial Component Placement
Parts:
- C1, C10, C14, C19, C2, C20, C3, C4, C6, C7, C8, C9, FB1, FB2, FB3, FB4, FB5, R10, R11, R13, R15, R16, R17, R18, R19, R20, R21, R22, R5, R6, R9, U2, U5, U7: moved to B.Cu
- moved J14 185.1 mm to (115.5, 129.8), turned to 90 degrees
- moved J11 170.6 mm to (115.1, 95.9), turned to 90 degrees
- moved JP4 168.0 mm to (181.9, 127.0)
- moved J23 164.2 mm to (190.8, 120.5)
- moved J8 163.4 mm to (173.4, 129.5)
- moved C17 162.3 mm to (181.9, 130.5)
- moved GND 160.1 mm to (181.6, 97.0), turned to 90 degrees
- moved JP2 158.3 mm to (177.2, 103.2), turned to 90 degrees
- moved +3V3 153.6 mm to (176.6, 97.0), turned to 90 degrees
- moved U5 153.0 mm to (172.8, 106.4)
- moved J12 152.5 mm to (114.3, 105.8)
- moved C14 149.0 mm to (178.4, 99.7)
- moved R11 148.7 mm to (178.3, 104.2), turned to -90 degrees
- moved JP3 147.2 mm to (162.2, 126.8)
- moved +5V 147.2 mm to (171.5, 97.0), turned to 90 degrees
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- renumbered TP2 to +3V3, TP1 to +5V, TP3 to GND
