File: _autosave-X17_Pi_Shield.kicad_pcb (KiCad board)
At the start: 2 copper layers, 85 x 56 mm, 89 parts, among them J1 BM04B-GHS-TBT, J10 BM04B-GHS-TBT, J11 BM04B-GHS-TBT, J12 Conn_01x05_Pin, J13 Conn_01x03_Pin, J2 BM02B-GHS-TBT, J20 Conn_01x02_Pin, J22 430450212, J23 430450612, J24 430450212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

Commit message: Layout
Routing:
- net GND: vias 0 -> 2
Changed lines of the file:
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@@
 		(net 5)
 	)
+	(via
+		(at 169 98)
+		(size 0.6)
+		(drill 0.3)
+		(layers "F.Cu" "B.Cu")
+		(free yes)
+		(net 5)
+	)
+	(via
+		(at 169.1 98.900003)
+		(size 0.6)
+		(drill 0.3)
+		(layers "F.Cu" "B.Cu")
+		(free yes)
+		(net 5)
+	)
 	(segment
 		(start 164.4729 104.4271)
@@
 	)
 	(segment
-		(start 170.234001 94.754)
-		(end 178.970526 94.754)
+		(start 179.795 85.04)
+		(end 179.795 85.448001)
 		(width 0.2)
 		(layer "F.Cu")
@@
 	)
 	(segment
-		(start 173.051471 111.5)
-		(end 175.880972 111.5)
+		(start 179.795 85.448001)
+		(end 179.218001 86.025)
 		(width 0.2)
 		(layer "F.Cu")
@@
 	)
 	(segment
-		(start 164.1228 128.21)
-		(end 164.8625 128.21)
+		(start 172.7 111.148529)
+		(end 173.051471 111.5)
 		(width 0.2)
 		(layer "F.Cu")
@@
 	)
 	(segment
-		(start 171.016722 124.425)
-		(end 165.3678 124.425)
+		(start 173.051471 111.5)
+		(end 175.880972 111.5)
 		(width 0.2)
 		(layer "F.Cu")
@@
 	)
 	(segment
-		(start 177.7075 117.734222)
-		(end 171.016722 124.425)
+		(start 175.880972 111.5)
+		(end 177.7075 113.326528)
+		(width 0.2)
+		(layer "F.Cu")
+		(net 54)
+	)
+	(segment
+		(start 177.7075 113.326528)
+		(end 177.7075 117.734222)
 		(width 0.2)
 		(layer "F.Cu")
@@
 	)
 	(segment
-		(start 181.35 85.04)
-		(end 174.549999 91.840001)
+		(start 164.1228 128.21)
+		(end 164.8625 128.21)
 		(width 0.2)
 		(layer "F.Cu")
@@
 	)
 	(segment
-		(start 180.704208 97.446)
-		(end 172.7 105.450208)
+		(start 172.7 105.450208)
+		(end 172.7 111.148529)
 		(width 0.2)
 		(layer "F.Cu")
@@
 	)
 	(segment
-		(start 178.970526 94.754)
-		(end 180.704208 96.487682)
+		(start 177.7075 117.734222)
+		(end 171.016722 124.425)
 		(width 0.2)
 		(layer "F.Cu")
@@
 	)
 	(segment
-		(start 180.704208 96.487682)
-		(end 180.704208 97.446)
+		(start 172.759999 91.840001)
+		(end 169.440002 91.840001)
+		(width 0.2)
+		(layer "F.Cu")
+		(net 54)
+	)
+	(segment
+		(start 180.704208 97.446)
+		(end 172.7 105.450208)
+		(width 0.2)
+		(layer "F.Cu")
+		(net 54)
+	)
+	(segment
+		(start 171.016722 124.425)
+		(end 165.3678 124.425)
 		(width 0.2)
 		(layer "F.Cu")
@@
 	)
 	(segment
-		(start 174.549999 91.840001)
-		(end 169.440002 91.840001)
+		(start 178.970526 94.754)
+		(end 180.704208 96.487682)
 		(width 0.2)
 		(layer "F.Cu")
@@
 	)
 	(segment
-		(start 163.4576 126.3352)
-		(end 163.4576 127.5448)
+		(start 179.218001 86.025)
+		(end 178.575 86.025)
 		(width 0.2)
 		(layer "F.Cu")
@@
 	)
 	(segment
-		(start 175.880972 111.5)
-		(end 177.7075 113.326528)
+		(start 170.234001 94.754)
+		(end 178.970526 94.754)
 		(width 0.2)
 		(layer "F.Cu")
@@
 	)
 	(segment
-		(start 172.7 111.148529)
-		(end 173.051471 111.5)
+		(start 181.35 85.04)
+		(end 179.795 85.04)
 		(width 0.2)
 		(layer "F.Cu")
@@
 	)
 	(segment
-		(start 172.7 105.450208)
-		(end 172.7 111.148529)
+		(start 163.4576 126.3352)
+		(end 163.4576 127.5448)
 		(width 0.2)
 		(layer "F.Cu")
@@
 	)
 	(segment
-		(start 177.7075 113.326528)
-		(end 177.7075 117.734222)
+		(start 180.704208 96.487682)
+		(end 180.704208 97.446)
+		(width 0.2)
+		(layer "F.Cu")
+		(net 54)
+	)
+	(segment
+		(start 178.575 86.025)
+		(end 172.759999 91.840001)
 		(width 0.2)
 		(layer "F.Cu")
@@
 		(fill yes
 			(thermal_gap 0.25)
-			(thermal_bridge_width 0.75)
+			(thermal_bridge_width 0.25)
 		)
 		(polygon
