File: _autosave-X17_Pi_Shield.kicad_pcb (KiCad board)
At the start: 4 copper layers, 85 x 56 mm, 89 parts, among them J1 BM04B-GHS-TBT, J10 BM04B-GHS-TBT, J11 BM04B-GHS-TBT, J12 Conn_01x05_Pin, J13 Conn_01x03_Pin, J2 BM02B-GHS-TBT, J20 Conn_01x02_Pin, J22 430450212, J23 430450612, J24 430450212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

Commit message: Hello Bruh
Routing:
- net Net-(U7-B): track 9.26 -> 24.3 mm, vias 0 -> 1
- net Net-(U7-VIO): track 0.00 -> 12.5 mm
- net Net-(U7-GND1): track 0.00 -> 12.3 mm
- net Net-(U7-VDD): track 0.00 -> 11.9 mm
- net Net-(U7-A): track 21.5 -> 29.9 mm
- net +3V3_TB: track 10.1 -> 15.4 mm
- net /Pi + IMU/TB_EN: track 0.00 -> 5.13 mm
- net GND_TB: track 15.6 -> 20.6 mm
- net /Pi + IMU/ISO_FLT: track 0.00 -> 4.02 mm
