File: power.kicad_sch (KiCad schematic)
At the start: 33 parts, among them J20 Conn_01x02_Pin, J8 UJC-HP-L-G-5-MSMT-TR, U2 TPS2117DRLR, U3 INA260AIPW, U9 AZ1117IH-3.3TRG1

Commit message: Finished Layout + Updated Capacitor Sizes for 150uF
Parts:
- C17, C5: footprint Capacitor_SMD:C_0603_1608Metric_Pad1.08x0.95mm_HandSolder -> Capacitor_SMD:C_1210_3225Metric_Pad1.33x2.70mm_HandSolder
Changed lines of the file:
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@@
 			)
 		)
-		(property "Footprint" "Capacitor_SMD:C_0603_1608Metric_Pad1.08x0.95mm_HandSolder"
+		(property "Footprint" "Capacitor_SMD:C_1210_3225Metric_Pad1.33x2.70mm_HandSolder"
 			(at 50.4952 161.29 0)
 			(effects
@@
 			)
 		)
-		(property "Footprint" "Capacitor_SMD:C_0603_1608Metric_Pad1.08x0.95mm_HandSolder"
+		(property "Footprint" "Capacitor_SMD:C_1210_3225Metric_Pad1.33x2.70mm_HandSolder"
 			(at 50.4952 187.96 0)
 			(effects
